File: Sensor.kicad_sch (KiCad schematic)
At the start: 12 parts, among them J2 Mini-DIN-3, J4 MD-30SM, U3 MCP6022-I/SN, U7 LM35CAZ

Commit message: gitignore
Parts:
- R11: value 100k 1% -> 75k 1%
Changed lines of the file:
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@@
 			)
 		)
-		(property "Value" "100k 1%"
+		(property "Value" "75k 1%"
 			(at 190.5 66.9544 90)
 			(effects
